File: PowerBus_24V/kicad/PowerBus_24V/PowerBus_24V.kicad_sch (KiCad schematic)
At the start: 0 parts

Commit message: changes
Parts:
- added J1: XT90PB-F, XT90PBF, symbol powerbus_24V:XT90PB-F
- added Q1: XT60_YELLOW, XT60, symbol powerbus_24V:XT60_YELLOW
