File: Gen1.5_PCB_draft/hardware/_restore_backup_2026-08-18T14-36-23-687/Gen1.5_PCB.kicad_sch (KiCad schematic)
At the start: 33 parts, among them IC1 TJA1050T, J1 Enc1, J10 jumper2, J11 jumper4, J12 Enc2, J13 Enc3, J14 Enc4, J15 Enc5, J16 Enc6, J17 jumper6, J2 Booster, J4 jumper1, J5 Roboclaw1, J6 Roboclaw2, J7 Roboclaw3, J8 jumper3, J9 jumper5, U1 ESP32-P4-ETH, U2 4754, U8 level shifter

Commit message: made whole pcb
Parts:
- removed J2: Booster, Gen1.5_PCB:booster headers, symbol Connector_Generic:Conn_01x04
- added J3: Booster, symbol Connector_Generic:Conn_01x03
- C19: footprint Gen1.5_PCB:CAP_0.1uF_50V -> CAN_test_board:CAPC2012X145N
- IC1: footprint Gen1.5_PCB:TJA1050T -> CAN_test_board:TJA1050T
- U1: footprint Gen1.5_PCB:MODULE_ESP32-P4-ETH -> ESP32-P4-ETH:MODULE_ESP32-P4-ETH
- U8: footprint Gen1.5_PCB:SOT95P280X145-5N -> CAN_test_board:SOT95P280X145-5N
Connections:
- net 10V: now also J3.VCC
- net 5V: now also J3.Vin
- net CS1: now also J1.4 (Pin_4); no longer J15.4 (Pin_4)
- net CS3: now also J13.4 (Pin_4); no longer J16.4 (Pin_4)
- net CS4: now also J14.4 (Pin_4); no longer J13.4 (Pin_4)
- net CS5: now also J15.4 (Pin_4); no longer J1.4 (Pin_4)
- net CS6: now also J16.4 (Pin_4); no longer J14.4 (Pin_4)
- net GND: now also J3.GND
- net MOSI: now reaches U1.27 (GPIO27)
- no-connect marks 18 -> 16
