File: Gen1.5_PCB_draft/hardware/_restore_backup_2026-08-18T15-47-37-212/Gen1.5_PCB.kicad_sch (KiCad schematic)
At the start: 33 parts, among them IC1 TJA1050T, J1 Enc1, J10 jumper2, J11 jumper4, J12 Enc2, J13 Enc3, J14 Enc4, J15 Enc5, J16 Enc6, J17 jumper6, J2 Booster, J4 jumper1, J5 Roboclaw1, J6 Roboclaw2, J7 Roboclaw3, J8 jumper3, J9 jumper5, U1 ESP32-P4-ETH, U2 4754, U8 level shifter

Commit message: made whole pcb
Connections:
- net MOSI: now reaches U1.27 (GPIO27)
- no-connect marks 18 -> 17
Changed lines of the file:
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@@
-	)
-	(no_connect
-		(at 25.4 171.45)
 	)
 	(no_connect
@@
 		(effects
 			(font
+				(size 1.27 1.27)
+			)
+			(justify right bottom)
+		)
+	)
+	(label "MOSI"
+		(at 25.4 171.45 180)
+		(effects
+			(font
