File: Gen1.5_PCB_draft/hardware/Gen1.5_PCB.kicad_sch (KiCad schematic)
At the start: 33 parts, among them IC1 TJA1050T, J1 Enc1, J10 jumper2, J11 jumper4, J12 Enc2, J13 Enc3, J14 Enc4, J15 Enc5, J16 Enc6, J17 jumper6, J2 Booster, J4 jumper1, J5 Roboclaw1, J6 Roboclaw2, J7 Roboclaw3, J8 jumper3, J9 jumper5, U1 ESP32-P4-ETH, U2 4754, U8 level shifter

Commit message: added correct lcsc for decoup caps and amps and edited silkscreen labels
Parts:
- C1, C18: LCSC C127833 -> C85858
- C19: LCSC (none) -> C85858
- U8: LCSC (none) -> C23654
Changed lines of the file:
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@@
 			)
 		)
+		(property "LCSC" "C85858"
+			(at 252.73 38.1 0)
+			(hide yes)
+			(show_name no)
+			(do_not_autoplace no)
+			(effects
+				(font
+					(size 1.27 1.27)
+				)
+			)
+		)
 		(pin "2"
 		)
@@
 			)
 		)
-		(property "LCSC" "C127833"
+		(property "LCSC" "C85858"
 			(at 99.06 138.43 0)
 			(hide yes)
@@
 			)
 		)
+		(property "LCSC" "C23654"
+			(at 226.06 52.07 0)
+			(show_name no)
+			(do_not_autoplace no)
+			(effects
+				(font
+					(size 1.27 1.27)
+				)
+			)
+		)
 		(pin "3"
 		)
@@
 			)
 		)
-		(property "LCSC" "C127833"
+		(property "LCSC" "C85858"
 			(at 185.42 91.44 0)
 			(hide yes)
