File: Gen1.5_PCB_draft/hardware/_restore_backup_2026-08-19T11-09-03-083/Gen1.5_PCB.kicad_pcb (KiCad board)
At the start: 4 copper layers, 74.8 x 101.5 mm, 67 parts, among them IC1 TJA1050T, J1 Enc1, J10 jumper2, J11 jumper4, J12 Enc2, J13 Enc3, J14 Enc4, J15 Enc5, J16 Enc6, J17 UART/CAN, J2 Booster, J4 UART/CAN, J5 MCP1, J6 MCP2, J7 MCP3, J8 UART/CAN, J9 jumper5, P2 LC1, P3 LC2, P4 LC3, P5 LC4, U1 ESP32-P4-ETH, U10 INA118U_2K5, U11 INA118U_2K5, U12 INA118U_2K5, U2 4754, U4 REF2033QDDCRQ1, U8 level shifter, U9 INA118U_2K5

Commit message: fixed sch according to last DR
Parts:
- J17: value UART/CAN -> jumper6
- J4: value UART/CAN -> jumper1
- J5: value MCP1 -> Roboclaw1
- J6: value MCP2 -> Roboclaw2
- J7: value MCP3 -> Roboclaw3
- J8: value UART/CAN -> jumper3
- P2: value LC1 -> loadcell 1
- P3: value LC2 -> loadcell 2
- P4: value LC3 -> loadcell 3
- P5: value LC4 -> loadcell 4
Routing:
- net 10V: track 140.5 -> 133.1 mm
- net /MISO: track 95.6 -> 91.3 mm
- net /SCL: track 30.0 -> 28.3 mm
- net /5V: track 51.6 -> 52.7 mm
- net /CANL: track 101.1 -> 100.1 mm
- net /CAN TX: track 66.5 -> 65.8 mm
- net Net-(J6-Pin_3): track 16.6 -> 16.0 mm
- net GND: vias 9 -> 6
