File: Gen1.5_powerbus/hardware/Gen1.5_powerbus.kicad_sch (KiCad schematic)
At the start: 0 parts

Commit message: added power and ground connectins
Parts:
- added J1: Battery, symbol Connector_Generic:Conn_01x02
- added J10: conn9, symbol Connector_Generic:Conn_01x02
- added J11: conn10, symbol Connector_Generic:Conn_01x02
- added J12: conn11, symbol Connector_Generic:Conn_01x02
- added J13: conn12, symbol Connector_Generic:Conn_01x02
- added J2: conn1, symbol Connector_Generic:Conn_01x02
- added J3: conn2, symbol Connector_Generic:Conn_01x02
- added J4: conn3, symbol Connector_Generic:Conn_01x02
- added J5: conn4, symbol Connector_Generic:Conn_01x02
- added J6: conn5, symbol Connector_Generic:Conn_01x02
- added J7: conn6, symbol Connector_Generic:Conn_01x02
- added J8: conn7, symbol Connector_Generic:Conn_01x02
- added J9: conn8, symbol Connector_Generic:Conn_01x02
Connections:
- new net V+: J1.1 (Pin_1), J10.1 (Pin_1), J11.1 (Pin_1), J12.1 (Pin_1), J13.1 (Pin_1), J2.1 (Pin_1), J3.1 (Pin_1), J4.1 (Pin_1), J5.1 (Pin_1), J6.1 (Pin_1), J7.1 (Pin_1), J8.1 (Pin_1), J9.1 (Pin_1)
- new net V-: J1.2 (Pin_2), J10.2 (Pin_2), J11.2 (Pin_2), J12.2 (Pin_2), J13.2 (Pin_2), J2.2 (Pin_2), J3.2 (Pin_2), J4.2 (Pin_2), J5.2 (Pin_2), J6.2 (Pin_2), J7.2 (Pin_2), J8.2 (Pin_2), J9.2 (Pin_2)
